File: adapter_board/pico_adapter.kicad_sch (KiCad schematic)
At the start: 2 parts, among them J1 Conn_02x05_Odd_Even, U1 Pico

Commit message: Add silkscreen connector pin numbers
This also updates to the latest version of KiCad, changes the default
page size to US letter and adds some details to the title block.  No
electrical changes were made.

Signed-off-by: Ed Beroset <beroset@ieee.org>
Parts:
- J1: footprint (none) -> Connector_PinHeader_2.00mm:PinHeader_2x05_P2.00mm_Vertical_SMD
Other:
- title: (none) -> pico-puller adapter board
Changed lines of the file:
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@@
-(kicad_sch (version 20211123) (generator eeschema)
-  (paper "A4")
+(kicad_sch (version 20230121) (generator eeschema)
+  (paper "USLetter")
+  (title_block
+    (title "pico-puller adapter board")
+    (date "2024-03-30")
+    (rev "1.2")
+    (comment 1 "E. Beroset")
+  )
   (junction (at 133.35 91.44) (diameter 0) (color 0 0 0 0)
   )
@@
   )
   (wire (pts (xy 160.02 91.44) (xy 166.37 91.44))
-    (stroke (width 0) (type default) (color 0 0 0 0))
+    (stroke (width 0) (type default))
   )
   (wire (pts (xy 133.35 86.36) (xy 147.32 86.36))
-    (stroke (width 0) (type default) (color 0 0 0 0))
+    (stroke (width 0) (type default))
   )
   (wire (pts (xy 161.29 96.52) (xy 160.02 96.52))
-    (stroke (width 0) (type default) (color 0 0 0 0))
+    (stroke (width 0) (type default))
   )
   (wire (pts (xy 133.35 91.44) (xy 133.35 86.36))
-    (stroke (width 0) (type default) (color 0 0 0 0))
+    (stroke (width 0) (type default))
   )
   (wire (pts (xy 115.57 82.55) (xy 133.35 82.55))
-    (stroke (width 0) (type default) (color 0 0 0 0))
+    (stroke (width 0) (type default))
   )
   (wire (pts (xy 171.45 105.41) (xy 171.45 86.36))
-    (stroke (width 0) (type default) (color 0 0 0 0))
+    (stroke (width 0) (type default))
   )
   (wire (pts (xy 160.02 88.9) (xy 168.91 88.9))
-    (stroke (width 0) (type default) (color 0 0 0 0))
+    (stroke (width 0) (type default))
   )
   (wire (pts (xy 142.24 102.87) (xy 142.24 115.57))
-    (stroke (width 0) (type default) (color 0 0 0 0))
+    (stroke (width 0) (type default))
   )
   (wire (pts (xy 147.32 93.98) (xy 142.24 93.98))
-    (stroke (width 0) (type default) (color 0 0 0 0))
+    (stroke (width 0) (type default))
   )
   (wire (pts (xy 160.02 93.98) (xy 163.83 93.98))
-    (stroke (width 0) (type default) (color 0 0 0 0))
+    (stroke (width 0) (type default))
   )
   (wire (pts (xy 129.54 88.9) (xy 129.54 113.03))
-    (stroke (width 0) (type default) (color 0 0 0 0))
+    (stroke (width 0) (type default))
   )
   (wire (pts (xy 168.91 88.9) (xy 168.91 110.49))
-    (stroke (width 0) (type default) (color 0 0 0 0))
+    (stroke (width 0) (type default))
   )
   (wire (pts (xy 168.91 110.49) (xy 115.57 110.49))
-    (stroke (width 0) (type default) (color 0 0 0 0))
+    (stroke (width 0) (type default))
   )
   (wire (pts (xy 147.32 96.52) (xy 133.35 96.52))
-    (stroke (width 0) (type default) (color 0 0 0 0))
+    (stroke (width 0) (type default))
   )
   (wire (pts (xy 161.29 107.95) (xy 161.29 96.52))
-    (stroke (width 0) (type default) (color 0 0 0 0))
+    (stroke (width 0) (type default))
   )
   (wire (pts (xy 115.57 102.87) (xy 142.24 102.87))
-    (stroke (width 0) (type default) (color 0 0 0 0))
+    (stroke (width 0) (type default))
   )
   (wire (pts (xy 115.57 107.95) (xy 161.29 107.95))
-    (stroke (width 0) (type default) (color 0 0 0 0))
+    (stroke (width 0) (type default))
   )
   (wire (pts (xy 166.37 115.57) (xy 142.24 115.57))
-    (stroke (width 0) (type default) (color 0 0 0 0))
+    (stroke (width 0) (type default))
   )
   (wire (pts (xy 147.32 88.9) (xy 129.54 88.9))
-    (stroke (width 0) (type default) (color 0 0 0 0))
+    (stroke (width 0) (type default))
   )
   (wire (pts (xy 129.54 113.03) (xy 115.57 113.03))
-    (stroke (width 0) (type default) (color 0 0 0 0))
+    (stroke (width 0) (type default))
   )
   (wire (pts (xy 133.35 96.52) (xy 133.35 91.44))
-    (stroke (width 0) (type default) (color 0 0 0 0))
+    (stroke (width 0) (type default))
   )
   (wire (pts (xy 133.35 82.55) (xy 133.35 86.36))
-    (stroke (width 0) (type default) (color 0 0 0 0))
+    (stroke (width 0) (type default))
   )
   (wire (pts (xy 115.57 105.41) (xy 171.45 105.41))
-    (stroke (width 0) (type default) (color 0 0 0 0))
+    (stroke (width 0) (type default))
   )
   (wire (pts (xy 163.83 93.98) (xy 163.83 100.33))
-    (stroke (width 0) (type default) (color 0 0 0 0))
+    (stroke (width 0) (type default))
   )
   (wire (pts (xy 142.24 93.98) (xy 142.24 102.87))
-    (stroke (width 0) (type default) (color 0 0 0 0))
+    (stroke (width 0) (type default))
   )
   (wire (pts (xy 171.45 86.36) (xy 160.02 86.36))
-    (stroke (width 0) (type default) (color 0 0 0 0))
+    (stroke (width 0) (type default))
   )
   (wire (pts (xy 166.37 91.44) (xy 166.37 115.57))
-    (stroke (width 0) (type default) (color 0 0 0 0))
+    (stroke (width 0) (type default))
   )
   (wire (pts (xy 163.83 100.33) (xy 115.57 100.33))
-    (stroke (width 0) (type default) (color 0 0 0 0))
+    (stroke (width 0) (type default))
   )
   (wire (pts (xy 133.35 91.44) (xy 147.32 91.44))
-    (stroke (width 0) (type default) (color 0 0 0 0))
+    (stroke (width 0) (type default))
   )
   (symbol (lib_id "Connector_Generic:Conn_02x05_Odd_Even") (at 152.4 91.44 0) (unit 1)
-    (in_bom yes) (on_board yes) (fields_autoplaced)
-    (property "Reference" "J1" (id 0) (at 153.67 80.01 0))
-    (property "Value" "Conn_02x05_Odd_Even" (id 1) (at 153.67 82.55 0))
-    (property "Footprint" "" (id 2) (at 152.4 91.44 0)
-      (effects (font (size 1.27 1.27)) hide)
-    )
-    (property "Datasheet" "~" (id 3) (at 152.4 91.44 0)
+    (in_bom yes) (on_board yes) (dnp no) (fields_autoplaced)
+    (property "Reference" "J1" (at 153.67 80.01 0)
+      (effects (font (size 1.27 1.27)))
+    )
+    (property "Value" "Conn_02x05_Odd_Even" (at 153.67 82.55 0)
+      (effects (font (size 1.27 1.27)))
+    )
+    (property "Footprint" "Connector_PinHeader_2.00mm:PinHeader_2x05_P2.00mm_Vertical_SMD" (at 152.4 91.44 0)
+      (effects (font (size 1.27 1.27)) hide)
+    )
+    (property "Datasheet" "~" (at 152.4 91.44 0)
       (effects (font (size 1.27 1.27)) hide)
     )
@@
     (pin "8")
     (pin "9")
+    (instances
+      (project "pico_adapter"
+        (path "/e63e39d7-6ac0-4ffd-8aa3-1841a4541b55"
+          (reference "J1") (unit 1)
+        )
+      )
+    )
   )
   (symbol (lib_id "MCU_RaspberryPi_and_Boards:Pico") (at 97.79 96.52 0) (unit 1)
-    (in_bom yes) (on_board yes) (fields_autoplaced)
-    (property "Reference" "U1" (id 0) (at 97.79 64.77 0))
-    (property "Value" "Pico" (id 1) (at 97.79 67.31 0))
-    (property "Footprint" "MCU_RaspberryPi_and_Boards:RPi_Pico_SMD_TH" (id 2) (at 97.79 96.52 90)
-      (effects (font (size 1.27 1.27)) hide)
-    )
-    (property "Datasheet" "" (id 3) (at 97.79 96.52 0)
+    (in_bom yes) (on_board yes) (dnp no) (fields_autoplaced)
+    (property "Reference" "U1" (at 97.79 64.77 0)
+      (effects (font (size 1.27 1.27)))
+    )
+    (property "Value" "Pico" (at 97.79 67.31 0)
+      (effects (font (size 1.27 1.27)))
+    )
+    (property "Footprint" "MCU_RaspberryPi_and_Boards:RPi_Pico_SMD_TH" (at 97.79 96.52 90)
+      (effects (font (size 1.27 1.27)) hide)
+    )
+    (property "Datasheet" "" (at 97.79 96.52 0)
       (effects (font (size 1.27 1.27)) hide)
     )
@@
     (pin "8")
     (pin "9")
+    (instances
+      (project "pico_adapter"
+        (path "/e63e39d7-6ac0-4ffd-8aa3-1841a4541b55"
+          (reference "U1") (unit 1)
+        )
+      )
+    )
   )
   (sheet_instances
     (path "/" (page "1"))
   )
-  (symbol_instances
-    (path "/83c43cd1-eea8-49b2-b3d7-28c19a42f1d6"
-      (reference "J1") (unit 1) (value "Conn_02x05_Odd_Even") (footprint "Connector_PinHeader_2.00mm:PinHeader_2x05_P2.00mm_Vertical_SMD")
-    )
-    (path "/a345bc54-2446-47f4-bcd1-2daf3693d5ce"
-      (reference "U1") (unit 1) (value "Pico") (footprint "MCU_RaspberryPi_and_Boards:RPi_Pico_SMD_TH")
-    )
-  )
 )
